File: CAD/KiCad/electronic box/electronic box.kicad_sch (KiCad schematic)
At the start: 55 parts, among them J1 DA15_Socket_MountingHoles, J2 Jack-DC, J5 DA15_Socket_MountingHoles, J6 Conn_02x03_Counter_Clockwise, J7 Conn_01x03

Commit message: Redesign main PCB.
Parts:
- removed female1/audio/testpoint1, female1/neopixel/testpoint1, female2/audio/testpoint1, female2/neopixel/testpoint1, female3/audio/testpoint1, female3/neopixel/testpoint1, male1/audio/testpoint1, male1/neopixel/testpoint1, male2/audio/testpoint1, male2/neopixel/testpoint1: Conn_01x01, Connector_PinHeader_1.00mm:PinHeader_1x01_P1.00mm_Vertical, symbol Connector_Generic:Conn_01x01
- removed female1/microphone/bridge1, female1/photosensor/bridge1, female2/microphone/bridge1, female2/photosensor/bridge1, female3/microphone/bridge1, female3/photosensor/bridge1, male1/microphone/bridge1, male1/photosensor/bridge1, male1/photosensor/bridge2, male1/photosensor/bridge3, male1/photosensor/bridge4, male2/microphone/bridge1, male2/photosensor/bridge1, male2/photosensor/bridge2, male2/photosensor/bridge3, male2/photosensor/bridge4: Conn_01x01, Connector_PinHeader_1.00mm:PinHeader_1x02_P1.00mm_Vertical, symbol Connector_Generic:Conn_01x02
- added J10, J8: Conn_01x08, Connector_PinHeader_2.54mm:PinHeader_1x08_P2.54mm_Vertical, symbol Connector_Generic:Conn_01x08
- added J11, J12: Conn_02x08_Odd_Even, Connector_PinHeader_2.54mm:PinHeader_2x08_P2.54mm_Vertical, symbol Connector_Generic:Conn_02x08_Odd_Even
- added J13, J14, J15, J16: Conn_01x02, Connector_PinHeader_2.54mm:PinHeader_1x02_P2.54mm_Vertical, symbol Connector_Generic:Conn_01x02
- added J3: Conn_01x06, Connector_PinHeader_2.54mm:PinHeader_1x08_P2.54mm_Vertical, symbol Connector_Generic:Conn_01x08
- added J4: Conn_01x10, Connector_PinHeader_2.54mm:PinHeader_1x10_P2.54mm_Vertical, symbol Connector_Generic:Conn_01x10
- added J9: Conn_02x18_Odd_Even, Connector_PinHeader_2.54mm:PinHeader_2x18_P2.54mm_Vertical, symbol Connector_Generic:Conn_02x18_Odd_Even
- added Q1, Q2: BC557, Package_TO_SOT_THT:TO-92_Inline, symbol Transistor_BJT:BC557
- added R1, R2: 150, Resistor_THT:R_Axial_DIN0207_L6.3mm_D2.5mm_P10.16mm_Horizontal, symbol Device:R
- added R3, R4: 10k, Resistor_THT:R_Axial_DIN0207_L6.3mm_D2.5mm_P10.16mm_Horizontal, symbol Device:R
- Extra1, Extra2: footprint Connector_PinHeader_1.00mm:PinHeader_1x06_P1.00mm_Vertical -> Connector_PinHeader_2.54mm:PinHeader_1x06_P2.54mm_Vertical
- J6: footprint Connector_PinHeader_2.54mm:PinHeader_2x03_P2.54mm_Vertical -> custom1:screw brigde
- female1/speaker/testpoint1, female2/speaker/testpoint1, female3/speaker/testpoint1, male1/speaker/testpoint1, male2/speaker/testpoint1: footprint Connector_PinHeader_1.00mm:PinHeader_1x02_P1.00mm_Vertical -> Connector_PinHeader_2.54mm:PinHeader_1x02_P2.54mm_Vertical
Connections:
- net male1/spearker - is gone; now on net male1/speaker -/out: B-J4.2, male1/amp1.2 (out_-)
- net +5V: now also Q1.3 (E), Q2.3 (E)
- net GND: now also A1.GND1 (GND), J4.4 (Pin_4); no longer A1.GND2 (GND)
- net female1/audio: now also J4.7 (Pin_7)
- net female1/microphone/1: now also J11.1 (Pin_1)
- net female1/microphone/2: now also J11.2 (Pin_2)
- net female1/neopixel: now also J8.2 (Pin_2)
- net female1/photosensor/1: now also J11.11 (Pin_11)
- net female1/photosensor/2: now also J11.12 (Pin_12)
- net female2/audio: now also J4.6 (Pin_6)
- net female2/microphone/1: now also J11.3 (Pin_3)
- net female2/microphone/2: now also J11.4 (Pin_4)
- net female2/neopixel: now also J8.1 (Pin_1)
- net female2/photosensor/1: now also J11.13 (Pin_13)
- net female2/photosensor/2: now also J11.14 (Pin_14)
- net female3/audio: now also J4.5 (Pin_5)
- net female3/microphone/1: now also J11.5 (Pin_5)
- net female3/microphone/2: now also J11.6 (Pin_6)
- net female3/neopixel: now also J4.10 (Pin_10)
- net female3/photosensor/1: now also J11.15 (Pin_15)
- net female3/photosensor/2: now also J11.16 (Pin_16)
- net male1/audio: now also J9.33 (Pin_33)
- net male1/bar neopixel: now also A1.D5, J8.3 (Pin_3)
- net male1/microphone/1: now also J11.7 (Pin_7)
- net male1/microphone/2: now also J11.8 (Pin_8)
- net male1/neopixel: now also J4.9 (Pin_9)
- net male1/photosensor/A/1: now also J12.1 (Pin_1)
- net male1/photosensor/A/2: now also J12.2 (Pin_2)
- net male1/photosensor/B/1: now also J12.3 (Pin_3)
- net male1/photosensor/B/2: now also J12.4 (Pin_4)
- net male1/photosensor/C/1: now also J12.5 (Pin_5)
- net male1/photosensor/C/2: now also J12.6 (Pin_6)
- net male1/photosensor/D/1: now also J12.7 (Pin_7)
- net male1/photosensor/D/2: now also J12.8 (Pin_8)
- net male1/speaker +/out: now also male1/amp1.1 (out_+)
- net male1/state LED: now also R1.2
- net male2/audio: now also J9.34 (Pin_34)
- net male2/bar neopixel: now also A1.D4, J8.4 (Pin_4)
- net male2/microphone/1: now also J11.9 (Pin_9)
- net male2/microphone/2: now also J11.10 (Pin_10)
- net male2/neopixel: now also J4.8 (Pin_8)
- net male2/photosensor/A/1: now also J12.9 (Pin_9)
- net male2/photosensor/A/2: now also J12.10 (Pin_10)
- net male2/photosensor/B/1: now also J12.11 (Pin_11)
- net male2/photosensor/B/2: now also J12.12 (Pin_12)
- net male2/photosensor/C/1: now also J12.13 (Pin_13)
- net male2/photosensor/C/2: now also J12.14 (Pin_14)
- net male2/photosensor/D/1: now also J12.15 (Pin_15)
- net male2/photosensor/D/2: now also J12.16 (Pin_16)
- net male2/speaker +/out: no longer male1/amp1.1 (out_+)
- net male2/state LED: now also R2.2
- net +3.3V: now reaches A1.3V3 (3.3V)
- net +3.3V: now also J3.4 (Pin_4)
- net 5V1: now reaches A1.5V1 (5V)
- net 5V1: now also J3.5 (Pin_5)
- net 5V3: now reaches A1.5V3 (5V)
- net 5V3: now also J9.35 (Pin_35)
- net 5V4: now reaches A1.5V4 (5V)
- net 5V4: now also J9.36 (Pin_36)
- net AREF: now reaches A1.AREF
- net AREF: now also J4.3 (Pin_3)
- net D0: now reaches A1.D0 (D0/RX0)
- net D0: now also J8.8 (Pin_8)
- net D1: now reaches A1.D1 (D1/TX0)
- net D1: now also J8.7 (Pin_7)
- net D14: now reaches A1.D14 (D14/TX3)
- net D14: now also J10.1 (Pin_1)
- net D15: now reaches A1.D15 (D15/RX3)
- net D15: now also J10.2 (Pin_2)
- net D16: now reaches A1.D16 (D16/TX2)
- net D16: now also J10.3 (Pin_3)
- net D17: now reaches A1.D17 (D17/RX2)
- net D17: now also J10.4 (Pin_4)
- net D18: now reaches A1.D18 (D18/TX1)
- net D18: now also J10.5 (Pin_5)
- net D19: now reaches A1.D19 (D19/RX1)
- net D19: now also J10.6 (Pin_6)
- net D2: now reaches A1.D2 (D2_INT0)
- net D2: now also J8.6 (Pin_6)
- net D20: now reaches A1.D20 (D20/SDA)
- net D20: now also J10.7 (Pin_7)
- net D21: now reaches A1.D21 (D21/SCL)
- net D21: now also J10.8 (Pin_8)
- net D24: now reaches A1.D24
- net D24: now also J9.31 (Pin_31), R3.1
- net D25: now reaches A1.D25
- net D25: now also J9.32 (Pin_32), R4.1
- net D26: now reaches A1.D26
- net D26: now also J9.29 (Pin_29)
- net D27: now reaches A1.D27
- net D27: now also J9.30 (Pin_30)
- net D28: now reaches A1.D28
- net D28: now also J9.27 (Pin_27)
- net D29: now reaches A1.D29
- net D29: now also J9.28 (Pin_28)
- net D3: now reaches A1.D3 (D3_INT1)
- net D3: now also J8.5 (Pin_5)
- net D30: now reaches A1.D30
- net D30: now also J9.25 (Pin_25)
- net D31: now reaches A1.D31
- net D31: now also J9.26 (Pin_26)
- net D32: now reaches A1.D32
- net D32: now also J9.23 (Pin_23)
- net D33: now reaches A1.D33
- net D33: now also J9.24 (Pin_24)
- net D34: now reaches A1.D34
- net D34: now also J9.21 (Pin_21)
- net D35: now reaches A1.D35
- net D35: now also J9.22 (Pin_22)
- net D36: now reaches A1.D36
- net D36: now also J9.19 (Pin_19)
- net D37: now reaches A1.D37
- net D37: now also J9.20 (Pin_20)
- net D38: now reaches A1.D38
- net D38: now also J9.17 (Pin_17)
- net D39: now reaches A1.D39
- net D39: now also J9.18 (Pin_18)
- net D40: now reaches A1.D40
- net D40: now also J9.15 (Pin_15)
- net D41: now reaches A1.D41
- net D41: now also J9.16 (Pin_16)
- net D42: now reaches A1.D42
- net D42: now also J9.13 (Pin_13)
- net D43: now reaches A1.D43
- net D43: now also J9.14 (Pin_14)
- net D44: now reaches A1.D44
- net D44: now also J9.11 (Pin_11)
- net D45: now reaches A1.D45
- net D45: now also J9.12 (Pin_12)
- net D46: now reaches A1.D46
- net D46: now also J9.9 (Pin_9)
- net D47: now reaches A1.D47
- net D47: now also J9.10 (Pin_10)
- net D48: now reaches A1.D48
- net D48: now also J9.7 (Pin_7)
- net D49: now reaches A1.D49
- net D49: now also J9.8 (Pin_8)
- net D50_MISO: now reaches A1.D50 (D50_MISO)
- net D50_MISO: now also J9.5 (Pin_5)
- net D51_MOSI: now reaches A1.D51 (D51_MOSI)
- net D51_MOSI: now also J9.6 (Pin_6)
- net D52_SCK: now reaches A1.D52 (D52_SCK)
- net D52_SCK: now also J9.3 (Pin_3)
- net D53_CS: now reaches A1.D53 (D53_CS)
- net D53_CS: now also J9.4 (Pin_4)
- net GND3: now reaches A1.GND3 (GND)
- net GND3: now also J3.7 (Pin_7)
- net GND5: now reaches A1.GND5 (GND)
- net GND5: now also J9.1 (Pin_1)
- net GND6: now reaches A1.GND6 (GND)
- net GND6: now also J9.2 (Pin_2)
- net IOREF: now reaches A1.IORF (IOREF)
- net IOREF: now also J3.2 (Pin_2)
- net RST1: now reaches A1.RST1 (RESET)
- net RST1: now also J3.3 (Pin_3)
- net SCL: now reaches A1.SCL
- net SCL: now also J4.1 (Pin_1)
- net SDA: now reaches A1.SDA
- net SDA: now also J4.2 (Pin_2)
- net at A1.VIN: now also J3.8 (Pin_8)
- new net: J15.1 (Pin_1), Q1.1 (C)
- new net: J15.2 (Pin_2), R1.1
- new net: J13.2 (Pin_2), Q1.2 (B)
- new net: J13.1 (Pin_1), R3.2
- new net: J14.1 (Pin_1), R4.2
- new net: J14.2 (Pin_2), Q2.2 (B)
- new net: J16.2 (Pin_2), R2.1
- new net: J16.1 (Pin_1), Q2.1 (C)
- new net GND2: A1.GND2 (GND), J3.6 (Pin_6)
- no-connect marks 0 -> 7
Other:
- moved on the sheet: dxl_data/testpoint1
