File: CAD/KiCad/shields/analyser-direct/analyser-direct.kicad_pcb (KiCad board)
At the start: 2 copper layers, 150 x 55 mm, 56 parts, among them U1 MCP6004-I/SL, U2 MCP6004-I/SL

Commit message: Remove shield identification and adopt the simplified connector and Teensy pin maps
Parts:
- removed CID1: 100nF, Shields:C_0603_1608Metric
- removed JSID1: WRITE ENABLE - OPEN, Shields:SolderJumper-2_P1.3mm_Open_RoundedPad1.0x1.5mm
- removed RID1: 10K, Shields:R_0603_1608Metric
- removed UID1: M24C02-RMN6TP, Shields:SOIC-8_3.9x4.9mm_P1.27mm
- added TPG: AGND, Shields:TestPoint_Pad_D1.5mm, F.Cu at (180.0, 94.0)
- JA1: value ANALYSER - KEY 24 -> ANALYSER - KEY 22; footprint Shields:Socket_2x12_Key24 -> Shields:Socket_2x11_Key22
Connections:
- JA1 pad 19: shield/sda -> IOREF
- JA1 pad 20: shield/scl -> (no net)
- JA1 pad 21: IOREF -> +5V
Routing:
- net GND: track 148.4 -> 0.00 mm
- net shield/sda: track 143.3 -> 0.00 mm, vias 1 -> 0
- net shield/scl: track 141.2 -> 0.00 mm, vias 1 -> 0
- net IOREF: track 216.4 -> 184.5 mm, vias 9 -> 7
- net AGND: track 404.1 -> 435.0 mm, vias 12 -> 16
- net female1/microphone: track 130.4 -> 152.3 mm, vias 0 -> 1
- net id/wp: track 19.2 -> 0.00 mm, vias 2 -> 0
- net female3/analyser out: track 79.2 -> 93.9 mm, vias 2 -> 1
- net male1/analyser out: track 99.0 -> 111.2 mm, vias 2 -> 1
- net male2/analyser out: track 126.4 -> 134.9 mm, vias 1 -> 0
- net female2/analyser out: track 58.3 -> 62.7 mm, vias 1 -> 2
- net +5V: track 107.6 -> 108.6 mm
- removed copper zone on B.Cu, net AGND
Other:
- board text added: "1"
- board text added: "AGND"
- board text added: "ANA 0"
- board text added: "ANA 1"
- board text added: "ANA 2"
- board text added: "ANA 3"
- board text added: "ANA 4"
- board text added: "ANALYSER - DIRECT TO TEENSY - RAW SAMPLES"
- board text added: "BENCH MIC - GND 5V SIG"
- board text added: "CH0 F1"
- board text added: "CH1 F2"
- board text added: "CH2 F3"
- board text added: "CH3 M1"
- board text added: "CH4 M2"
- board text added: "HARNESS < CH0 > BENCH"
- board text added: "IOREF"
- board text added: "KEY <-"
- board text added: "UNPLUGGED MIC = 0 V"
- board text removed: "ANALYSER-DIRECT"

Commit message: Finish revised shield routing, printed identification and clean KiCad checks
Routing:
- added copper zone on B.Cu, net AGND
Changed lines of the file:
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@@
 		(descr "Physical top-view contact map; bottom mounted socket, blocked final cavity")
 		(property "Reference" "JA1"
-			(at 0 0 0)
+			(at 6 0 0)
 			(layer "F.SilkS")
 			(effects
@@
 			(size 1.7 1.7)
 			(drill 1)
-			(layers "*.Cu")
+			(layers "*.Cu" "*.Mask")
 			(remove_unused_layers no)
 			(net 9 "female1{slash}microphone")
@@
 			(size 1.7 1.7)
 			(drill 1)
-			(layers "*.Cu")
+			(layers "*.Cu" "*.Mask")
 			(remove_unused_layers no)
 			(net 2 "AGND")
@@
 			(size 1.7 1.7)
 			(drill 1)
-			(layers "*.Cu")
+			(layers "*.Cu" "*.Mask")
 			(remove_unused_layers no)
 			(net 14 "female2{slash}microphone")
@@
 			(size 1.7 1.7)
 			(drill 1)
-			(layers "*.Cu")
+			(layers "*.Cu" "*.Mask")
 			(remove_unused_layers no)
 			(net 2 "AGND")
@@
 			(size 1.7 1.7)
 			(drill 1)
-			(layers "*.Cu")
+			(layers "*.Cu" "*.Mask")
 			(remove_unused_layers no)
 			(net 19 "female3{slash}microphone")
@@
 			(size 1.7 1.7)
 			(drill 1)
-			(layers "*.Cu")
+			(layers "*.Cu" "*.Mask")
 			(remove_unused_layers no)
 			(net 2 "AGND")
@@
 			(size 1.7 1.7)
 			(drill 1)
-			(layers "*.Cu")
+			(layers "*.Cu" "*.Mask")
 			(remove_unused_layers no)
 			(net 24 "male1{slash}microphone")
@@
 			(size 1.7 1.7)
 			(drill 1)
-			(layers "*.Cu")
+			(layers "*.Cu" "*.Mask")
 			(remove_unused_layers no)
 			(net 2 "AGND")
@@
 			(size 1.7 1.7)
 			(drill 1)
-			(layers "*.Cu")
+			(layers "*.Cu" "*.Mask")
 			(remove_unused_layers no)
 			(net 29 "male2{slash}microphone")
@@
 			(size 1.7 1.7)
 			(drill 1)
-			(layers "*.Cu")
+			(layers "*.Cu" "*.Mask")
 			(remove_unused_layers no)
 			(net 2 "AGND")
@@
 			(size 1.7 1.7)
 			(drill 1)
-			(layers "*.Cu")
+			(layers "*.Cu" "*.Mask")
 			(remove_unused_layers no)
 			(net 6 "female1{slash}analyser out")
@@
 			(size 1.7 1.7)
 			(drill 1)
-			(layers "*.Cu")
+			(layers "*.Cu" "*.Mask")
 			(remove_unused_layers no)
 			(net 11 "female2{slash}analyser out")
@@
 			(size 1.7 1.7)
 			(drill 1)
-			(layers "*.Cu")
+			(layers "*.Cu" "*.Mask")
 			(remove_unused_layers no)
 			(net 16 "female3{slash}analyser out")
@@
 			(size 1.7 1.7)
 			(drill 1)
-			(layers "*.Cu")
+			(layers "*.Cu" "*.Mask")
 			(remove_unused_layers no)
 			(net 21 "male1{slash}analyser out")
@@
 			(size 1.7 1.7)
 			(drill 1)
-			(layers "*.Cu")
+			(layers "*.Cu" "*.Mask")
 			(remove_unused_layers no)
 			(net 26 "male2{slash}analyser out")
@@
 			(size 1.7 1.7)
 			(drill 1)
-			(layers "*.Cu")
+			(layers "*.Cu" "*.Mask")
 			(remove_unused_layers no)
 			(net 2 "AGND")
@@
 			(size 1.7 1.7)
 			(drill 1)
-			(layers "*.Cu")
+			(layers "*.Cu" "*.Mask")
 			(remove_unused_layers no)
 			(thermal_bridge_angle 45)
@@
 			(size 1.7 1.7)
 			(drill 1)
-			(layers "*.Cu")
+			(layers "*.Cu" "*.Mask")
 			(remove_unused_layers no)
 			(thermal_bridge_angle 45)
@@
 			(size 1.7 1.7)
 			(drill 1)
-			(layers "*.Cu")
+			(layers "*.Cu" "*.Mask")
 			(remove_unused_layers no)
 			(net 3 "IOREF")
@@
 			(size 1.7 1.7)
 			(drill 1)
-			(layers "*.Cu")
+			(layers "*.Cu" "*.Mask")
 			(remove_unused_layers no)
 			(thermal_bridge_angle 45)
@@
 			(size 1.7 1.7)
 			(drill 1)
-			(layers "*.Cu")
+			(layers "*.Cu" "*.Mask")
 			(remove_unused_layers no)
 			(net 1 "+5V")
@@
 		(layer "Edge.Cuts")
 	)
-	(gr_text "ANA 0"
-		(at 68 95 0)
+	(gr_text "CH0 F1"
+		(at 68 81 0)
 		(layer "F.SilkS")
 		(effects
 			(font
-				(size 0.8 0.8)
+				(size 0.9 0.9)
 				(thickness 0.12)
 			)
 		)
 	)
-	(gr_text "KEY <-"
-		(at 60 79.4 0)
+	(gr_text "HARNESS < CH0 > BENCH"
+		(at 164 83 0)
 		(layer "F.SilkS")
 		(effects
@@
 		)
 	)
-	(gr_text "CH0 F1"
-		(at 68 81 0)
+	(gr_text "KEY <-"
+		(at 60 79.4 0)
 		(layer "F.SilkS")
 		(effects
 			(font
-				(size 0.9 0.9)
+				(size 0.8 0.8)
 				(thickness 0.12)
 			)
 		)
 	)
-	(gr_text "ANALYSER - DIRECT TO TEENSY - RAW SAMPLES"
-		(at 123 52 0)
+	(gr_text "ANA 0"
+		(at 68 95 0)
 		(layer "F.SilkS")
 		(effects
 			(font
-				(size 1.2 1.2)
+				(size 0.8 0.8)
 				(thickness 0.12)
 			)
 		)
 	)
-	(gr_text "CH3 M1"
-		(at 134 81 0)
+	(gr_text "AGND"
+		(at 180 96 0)
 		(layer "F.SilkS")
 		(effects
 			(font
-				(size 0.9 0.9)
+				(size 0.8 0.8)
 				(thickness 0.12)
 			)
 		)
 	)
-	(gr_text "CH1 F2"
-		(at 90 81 0)
+	(gr_text "ANA 1"
+		(at 90 95 0)
 		(layer "F.SilkS")
 		(effects
 			(font
-				(size 0.9 0.9)
+				(size 0.8 0.8)
 				(thickness 0.12)
 			)
 		)
 	)
-	(gr_text "ANA 4"
-		(at 156 95 0)
+	(gr_text "IOREF"
+		(at 186 96 0)
 		(layer "F.SilkS")
 		(effects
@@
 		)
 	)
-	(gr_text "AGND"
-		(at 180 96 0)
+	(gr_text "ANA 4"
+		(at 156 95 0)
 		(layer "F.SilkS")
 		(effects
@@
 		)
 	)
-	(gr_text "BENCH MIC - GND 5V SIG"
-		(at 151 103 0)
+	(gr_text "CH2 F3"
+		(at 112 82.5 0)
 		(layer "F.SilkS")
 		(effects
 			(font
-				(size 0.8 0.8)
+				(size 0.9 0.9)
 				(thickness 0.12)
 			)
 		)
 	)
-	(gr_text "UNPLUGGED MIC = 0 V"
-		(at 123 99 0)
+	(gr_text "CH4 M2"
+		(at 156 81 0)
 		(layer "F.SilkS")
 		(effects
 			(font
-				(size 1 1)
+				(size 0.9 0.9)
 				(thickness 0.12)
 			)
 		)
 	)
-	(gr_text "CH4 M2"
-		(at 156 81 0)
+	(gr_text "CH1 F2"
+		(at 90 81 0)
 		(layer "F.SilkS")
 		(effects
@@
 		)
 	)
-	(gr_text "CH2 F3"
-		(at 112 82.5 0)
+	(gr_text "ANALYSER - DIRECT TO TEENSY - RAW SAMPLES"
+		(at 123 52 0)
 		(layer "F.SilkS")
 		(effects
 			(font
-				(size 0.9 0.9)
+				(size 1.2 1.2)
 				(thickness 0.12)
 			)
 		)
 	)
-	(gr_text "ANA 3"
-		(at 134 95 0)
+	(gr_text "ANA 2"
+		(at 112 95 0)
 		(layer "F.SilkS")
 		(effects
@@
 		)
 	)
-	(gr_text "IOREF"
-		(at 186 96 0)
+	(gr_text "ANA 3"
+		(at 134 95 0)
 		(layer "F.SilkS")
 		(effects
@@
 		)
 	)
-	(gr_text "ANA 1"
-		(at 90 95 0)
+	(gr_text "CH3 M1"
+		(at 134 81 0)
 		(layer "F.SilkS")
 		(effects
 			(font
-				(size 0.8 0.8)
+				(size 0.9 0.9)
 				(thickness 0.12)
 			)
 		)
 	)
-	(gr_text "HARNESS < CH0 > BENCH"
-		(at 164 83 0)
+	(gr_text "BENCH MIC - GND 5V SIG"
+		(at 151 103 0)
 		(layer "F.SilkS")
 		(effects
@@
 		)
 	)
-	(gr_text "ANA 2"
-		(at 112 95 0)
+	(gr_text "UNPLUGGED MIC = 0 V"
+		(at 123 99 0)
 		(layer "F.SilkS")
 		(effects
 			(font
-				(size 0.8 0.8)
+				(size 1 1)
 				(thickness 0.12)
 			)
@@
 		(net 33)
 	)
+	(zone
+		(net 2)
+		(net_name "AGND")
+		(layer "B.Cu")
+		(name "SH_RETURN")
+		(hatch edge 0.5)
+		(connect_pads yes
+			(clearance 0.25)
+		)
+		(min_thickness 0.2)
+		(filled_areas_thickness no)
+		(fill yes
+			(thermal_gap 0.5)
+			(thermal_bridge_width 0.5)
+		)
+		(polygon
+			(pts
+				(xy 50.45 50.45) (xy 199.55 50.45) (xy 199.55 104.55) (xy 50.45 104.55)
+			)
+		)
+	)
 	(embedded_fonts no)
