File: CAD/KiCad/shields/analyser-msgeq7/analyser-msgeq7-placed.kicad_pcb (KiCad board)
At the start: 2 copper layers, 150 x 55 mm, 59 parts, among them U1 MSGEQ7N, U2 MSGEQ7N, U3 MSGEQ7N, U4 MSGEQ7N, U5 MSGEQ7N

Commit message: Route the shield set and validate shared interfaces
Connections:
- JA1 pad 23: +5V -> (no net)

Commit message: Remove shield identification and adopt the simplified connector and Teensy pin maps
Parts:
- removed CID1: 100nF, Shields:C_0603_1608Metric
- removed JSID1: WRITE ENABLE - OPEN, Shields:SolderJumper-2_P1.3mm_Open_RoundedPad1.0x1.5mm
- removed RID1: 10K, Shields:R_0603_1608Metric
- removed UID1: M24C02-RMN6TP, Shields:SOIC-8_3.9x4.9mm_P1.27mm
- added TPG: AGND, Shields:TestPoint_Pad_D1.5mm, F.Cu at (183.0, 90.0)
- added TPI: IOREF, Shields:TestPoint_Pad_D1.5mm, F.Cu at (178.0, 90.0)
- JA1: value ANALYSER - KEY 24 -> ANALYSER - KEY 22; footprint Shields:Socket_2x12_Key24 -> Shields:Socket_2x11_Key22
Connections:
- JA1 pad 19: shield/sda -> IOREF
- JA1 pad 20: shield/scl -> (no net)
- JA1 pad 21: IOREF -> (no net)

Commit message: Route microphones directly to Teensy and remove the analyser buffer board
Parts:
- TPI: value IOREF -> MEGA_5V
Connections:
- net IOREF renamed MEGA_5V
Other:
- board text added: "1"
- board text added: "AGND"
- board text added: "ANA 0"
- board text added: "ANA 1"
- board text added: "ANA 2"
- board text added: "ANA 3"
- board text added: "ANA 4"
- board text added: "CH0 F1"
- board text added: "CH1 F2"
- board text added: "CH2 F3"
- board text added: "CH3 M1"
- board text added: "CH4 M2"
- board text added: "KEY <-"
- board text added: "MEGA 5V"
- board text added: "MSGEQ7 ANALYSER - MEGA ONLY"
- board text added: "OPEN UNLESS MEASURED"
- board text added: "REF - NEVER GROUND"
- board text added: "RESET"
- board text added: "STROBE"
- board text removed: "ANALYSER-MSGEQ7"
