File: CAD/KiCad/shields/analyser-msgeq7/female2.kicad_sch (KiCad schematic)
At the start: 10 parts, among them U4 MSGEQ7N

Commit message: Route microphones directly to Teensy and remove the analyser buffer board
Connections:
- net IOREF renamed MEGA_5V
Changed lines of the file:
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@@
 (kicad_sch (version 20250114) (generator "eeschema") (generator_version "9.0")
  (paper "A3")
-          (title_block (title "analyser-msgeq7 / female2") (date "2026-10-04") (rev "A-prototype")
+          (title_block (title "analyser-msgeq7 / female2") (date "2026-10-05") (rev "A-prototype")
             (company "Colloquy of Mobiles") (comment 1 "Prototype: verify harness polarity and sensor values before connection"))
           (text "COLLOQUY / ANALYSER-MSGEQ7 / FEMALE2" (at 15.24 15.24 0) (effects (font (size 2.032 2.032) (bold yes)) (justify left top)))
@@
 (instances (project "analyser-msgeq7" (path "/051aa90c-bb55-5623-9e53-94470bed9b3c/dc261c20-56d8-521f-a1cb-54128e0c60cf" (reference "U4") (unit 1)))))
 (wire (pts (xy 81.2800 66.0400) (xy 78.7400 66.0400)) (stroke (width 0) (type default)))
-(global_label "IOREF" (shape bidirectional) (at 78.7400 66.0400 180) (effects (font (size 0.95 0.95)) (justify right)) (property "Intersheetrefs" "${INTERSHEET_REFS}" (at 78.7400 66.0400 0) (effects (font (size 1.016 1.016))  (hide yes))))
+(global_label "MEGA_5V" (shape bidirectional) (at 78.7400 66.0400 180) (effects (font (size 0.95 0.95)) (justify right)) (property "Intersheetrefs" "${INTERSHEET_REFS}" (at 78.7400 66.0400 0) (effects (font (size 1.016 1.016))  (hide yes))))
 (wire (pts (xy 81.2800 71.1200) (xy 78.7400 71.1200)) (stroke (width 0) (type default)))
 (global_label "AGND" (shape bidirectional) (at 78.7400 71.1200 180) (effects (font (size 0.95 0.95)) (justify right)) (property "Intersheetrefs" "${INTERSHEET_REFS}" (at 78.7400 71.1200 0) (effects (font (size 1.016 1.016))  (hide yes))))
@@
 (instances (project "analyser-msgeq7" (path "/051aa90c-bb55-5623-9e53-94470bed9b3c/dc261c20-56d8-521f-a1cb-54128e0c60cf" (reference "R413") (unit 1)))))
 (wire (pts (xy 190.5000 154.9400) (xy 187.9600 154.9400)) (stroke (width 0) (type default)))
-(global_label "IOREF" (shape bidirectional) (at 187.9600 154.9400 180) (effects (font (size 0.95 0.95)) (justify right)) (property "Intersheetrefs" "${INTERSHEET_REFS}" (at 187.9600 154.9400 0) (effects (font (size 1.016 1.016))  (hide yes))))
+(global_label "MEGA_5V" (shape bidirectional) (at 187.9600 154.9400 180) (effects (font (size 0.95 0.95)) (justify right)) (property "Intersheetrefs" "${INTERSHEET_REFS}" (at 187.9600 154.9400 0) (effects (font (size 1.016 1.016))  (hide yes))))
 (wire (pts (xy 200.6600 154.9400) (xy 203.2000 154.9400)) (stroke (width 0) (type default)))
 (global_label "female2/oscillator" (shape bidirectional) (at 203.2000 154.9400 0) (effects (font (size 0.95 0.95)) (justify left)) (property "Intersheetrefs" "${INTERSHEET_REFS}" (at 203.2000 154.9400 0) (effects (font (size 1.016 1.016))  (hide yes))))
@@
 (instances (project "analyser-msgeq7" (path "/051aa90c-bb55-5623-9e53-94470bed9b3c/dc261c20-56d8-521f-a1cb-54128e0c60cf" (reference "C415") (unit 1)))))
 (wire (pts (xy 325.1200 180.3400) (xy 325.1200 177.8000)) (stroke (width 0) (type default)))
-(global_label "IOREF" (shape bidirectional) (at 325.1200 177.8000 0) (effects (font (size 0.95 0.95)) (justify left)) (property "Intersheetrefs" "${INTERSHEET_REFS}" (at 325.1200 177.8000 0) (effects (font (size 1.016 1.016))  (hide yes))))
+(global_label "MEGA_5V" (shape bidirectional) (at 325.1200 177.8000 0) (effects (font (size 0.95 0.95)) (justify left)) (property "Intersheetrefs" "${INTERSHEET_REFS}" (at 325.1200 177.8000 0) (effects (font (size 1.016 1.016))  (hide yes))))
 (wire (pts (xy 325.1200 190.5000) (xy 325.1200 193.0400)) (stroke (width 0) (type default)))
 (global_label "AGND" (shape bidirectional) (at 325.1200 193.0400 0) (effects (font (size 0.95 0.95)) (justify left)) (property "Intersheetrefs" "${INTERSHEET_REFS}" (at 325.1200 193.0400 0) (effects (font (size 1.016 1.016))  (hide yes))))
