File: CAD/KiCad/shields/teensy-adapter/mega.kicad_sch (KiCad schematic)
At the start: 1 part

Commit message: Route microphones directly to Teensy and remove the analyser buffer board
Connections:
- net analyser/reset: no longer names the net of JM1.D3
- net analyser/strobe: no longer names the net of JM1.D4
- net female1/analyser out: no longer names the net of JM1.A0
- net female2/analyser out: no longer names the net of JM1.A1
- net female3/analyser out: no longer names the net of JM1.A2
- net male1/analyser out: no longer names the net of JM1.A3
- net male2/analyser out: no longer names the net of JM1.A4
- no-connect marks 11 -> 18
Changed lines of the file:
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@@
 (kicad_sch (version 20250114) (generator "eeschema") (generator_version "9.0")
  (paper "A3")
-          (title_block (title "teensy-adapter / mega") (date "2026-10-04") (rev "A-prototype")
+          (title_block (title "teensy-adapter / mega") (date "2026-10-05") (rev "A-prototype")
             (company "Colloquy of Mobiles") (comment 1 "Prototype: verify harness polarity and sensor values before connection"))
           (text "COLLOQUY / TEENSY-ADAPTER / MEGA" (at 15.24 15.24 0) (effects (font (size 2.032 2.032) (bold yes)) (justify left top)))
@@
 (wire (pts (xy 121.9200 81.2800) (xy 124.4600 81.2800)) (stroke (width 0) (type default)))
 (global_label "male2/tone" (shape bidirectional) (at 124.4600 81.2800 0) (effects (font (size 0.95 0.95)) (justify left)) (property "Intersheetrefs" "${INTERSHEET_REFS}" (at 124.4600 81.2800 0) (effects (font (size 1.016 1.016))  (hide yes))))
-(wire (pts (xy 121.9200 86.3600) (xy 124.4600 86.3600)) (stroke (width 0) (type default)))
-(global_label "analyser/strobe" (shape bidirectional) (at 124.4600 86.3600 0) (effects (font (size 0.95 0.95)) (justify left)) (property "Intersheetrefs" "${INTERSHEET_REFS}" (at 124.4600 86.3600 0) (effects (font (size 1.016 1.016))  (hide yes))))
-(wire (pts (xy 121.9200 91.4400) (xy 124.4600 91.4400)) (stroke (width 0) (type default)))
-(global_label "analyser/reset" (shape bidirectional) (at 124.4600 91.4400 0) (effects (font (size 0.95 0.95)) (justify left)) (property "Intersheetrefs" "${INTERSHEET_REFS}" (at 124.4600 91.4400 0) (effects (font (size 1.016 1.016))  (hide yes))))
-(wire (pts (xy 121.9200 96.5200) (xy 124.4600 96.5200)) (stroke (width 0) (type default)))
-(global_label "female1/analyser out" (shape bidirectional) (at 124.4600 96.5200 0) (effects (font (size 0.95 0.95)) (justify left)) (property "Intersheetrefs" "${INTERSHEET_REFS}" (at 124.4600 96.5200 0) (effects (font (size 1.016 1.016))  (hide yes))))
-(wire (pts (xy 121.9200 101.6000) (xy 124.4600 101.6000)) (stroke (width 0) (type default)))
-(global_label "female2/analyser out" (shape bidirectional) (at 124.4600 101.6000 0) (effects (font (size 0.95 0.95)) (justify left)) (property "Intersheetrefs" "${INTERSHEET_REFS}" (at 124.4600 101.6000 0) (effects (font (size 1.016 1.016))  (hide yes))))
-(wire (pts (xy 121.9200 106.6800) (xy 124.4600 106.6800)) (stroke (width 0) (type default)))
-(global_label "female3/analyser out" (shape bidirectional) (at 124.4600 106.6800 0) (effects (font (size 0.95 0.95)) (justify left)) (property "Intersheetrefs" "${INTERSHEET_REFS}" (at 124.4600 106.6800 0) (effects (font (size 1.016 1.016))  (hide yes))))
-(wire (pts (xy 121.9200 111.7600) (xy 124.4600 111.7600)) (stroke (width 0) (type default)))
-(global_label "male1/analyser out" (shape bidirectional) (at 124.4600 111.7600 0) (effects (font (size 0.95 0.95)) (justify left)) (property "Intersheetrefs" "${INTERSHEET_REFS}" (at 124.4600 111.7600 0) (effects (font (size 1.016 1.016))  (hide yes))))
+(no_connect (at 121.9200 86.3600))
+(no_connect (at 121.9200 91.4400))
+(no_connect (at 121.9200 96.5200))
+(no_connect (at 121.9200 101.6000))
+(no_connect (at 121.9200 106.6800))
+(no_connect (at 121.9200 111.7600))
 (symbol (lib_id "Colloquy:JM1") (at 307.3400 83.8200 0) (unit 2) (exclude_from_sim no) (in_bom yes) (on_board yes) (dnp no)
 (property "Reference" "JM1" (at 307.3400 48.2600 0) (effects (font (size 1.016 1.016))  ))
@@
 (pin "D22")
 (instances (project "teensy-adapter" (path "/2a34184d-f581-57f8-88bf-73706d912fa4/f260262e-1c6d-5655-a113-171412ba1d71" (reference "JM1") (unit 2)))))
-(wire (pts (xy 287.0200 55.8800) (xy 284.4800 55.8800)) (stroke (width 0) (type default)))
-(global_label "male2/analyser out" (shape bidirectional) (at 284.4800 55.8800 180) (effects (font (size 0.95 0.95)) (justify right)) (property "Intersheetrefs" "${INTERSHEET_REFS}" (at 284.4800 55.8800 0) (effects (font (size 1.016 1.016))  (hide yes))))
+(no_connect (at 287.0200 55.8800))
 (wire (pts (xy 287.0200 60.9600) (xy 284.4800 60.9600)) (stroke (width 0) (type default)))
 (global_label "female1/neopixel/driven" (shape bidirectional) (at 284.4800 60.9600 180) (effects (font (size 0.95 0.95)) (justify right)) (property "Intersheetrefs" "${INTERSHEET_REFS}" (at 284.4800 60.9600 0) (effects (font (size 1.016 1.016))  (hide yes))))
