File: CAD/KiCad/shields/teensy-adapter/mega_2.kicad_sch (KiCad schematic)
At the start: 1 part

Commit message: Remove shield identification and adopt the simplified connector and Teensy pin maps
Connections:
- net shield/scl: no longer names the net of JM1.SCL
- net shield/sda: no longer names the net of JM1.SDA
- no-connect marks 30 -> 32
Changed lines of the file:
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@@
 (global_label "IOREF" (shape bidirectional) (at 284.4800 96.5200 180) (effects (font (size 0.95 0.95)) (justify right)) (property "Intersheetrefs" "${INTERSHEET_REFS}" (at 284.4800 96.5200 0) (effects (font (size 1.016 1.016))  (hide yes))))
 (no_connect (at 287.0200 101.6000))
-(wire (pts (xy 287.0200 106.6800) (xy 284.4800 106.6800)) (stroke (width 0) (type default)))
-(global_label "shield/scl" (shape bidirectional) (at 284.4800 106.6800 180) (effects (font (size 0.95 0.95)) (justify right)) (property "Intersheetrefs" "${INTERSHEET_REFS}" (at 284.4800 106.6800 0) (effects (font (size 1.016 1.016))  (hide yes))))
-(wire (pts (xy 287.0200 111.7600) (xy 284.4800 111.7600)) (stroke (width 0) (type default)))
-(global_label "shield/sda" (shape bidirectional) (at 284.4800 111.7600 180) (effects (font (size 0.95 0.95)) (justify right)) (property "Intersheetrefs" "${INTERSHEET_REFS}" (at 284.4800 111.7600 0) (effects (font (size 1.016 1.016))  (hide yes))))
+(no_connect (at 287.0200 106.6800))
+(no_connect (at 287.0200 111.7600))
 (no_connect (at 327.6600 83.8200))
           (embedded_fonts no))

Commit message: Route microphones directly to Teensy and remove the analyser buffer board
Connections:
- net female1/mic direct: now reaches JM1.D26
- net female2/mic direct: now reaches JM1.D27
- net female3/mic direct: now reaches JM1.D28
- net male1/mic direct: now reaches JM1.D29
- net male2/mic direct: now reaches JM1.D30
- net IOREF: no longer names the net of JM1.IORF
- no-connect marks 32 -> 28
Changed lines of the file:
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@@
 (kicad_sch (version 20250114) (generator "eeschema") (generator_version "9.0")
  (paper "A3")
-          (title_block (title "teensy-adapter / mega") (date "2026-10-04") (rev "A-prototype")
+          (title_block (title "teensy-adapter / mega") (date "2026-10-05") (rev "A-prototype")
             (company "Colloquy of Mobiles") (comment 1 "Prototype: verify harness polarity and sensor values before connection"))
           (text "COLLOQUY / TEENSY-ADAPTER / MEGA" (at 15.24 15.24 0) (effects (font (size 2.032 2.032) (bold yes)) (justify left top)))
@@
 (instances (project "teensy-adapter" (path "/2a34184d-f581-57f8-88bf-73706d912fa4/f260262e-1c6d-5655-a113-171412ba1d71" (reference "JM1") (unit 3)))))
 (no_connect (at 81.2800 55.8800))
-(no_connect (at 81.2800 60.9600))
-(no_connect (at 81.2800 66.0400))
-(no_connect (at 81.2800 71.1200))
-(no_connect (at 81.2800 76.2000))
-(no_connect (at 81.2800 81.2800))
+(wire (pts (xy 81.2800 60.9600) (xy 78.7400 60.9600)) (stroke (width 0) (type default)))
+(global_label "female1/mic direct" (shape bidirectional) (at 78.7400 60.9600 180) (effects (font (size 0.95 0.95)) (justify right)) (property "Intersheetrefs" "${INTERSHEET_REFS}" (at 78.7400 60.9600 0) (effects (font (size 1.016 1.016))  (hide yes))))
+(wire (pts (xy 81.2800 66.0400) (xy 78.7400 66.0400)) (stroke (width 0) (type default)))
+(global_label "female2/mic direct" (shape bidirectional) (at 78.7400 66.0400 180) (effects (font (size 0.95 0.95)) (justify right)) (property "Intersheetrefs" "${INTERSHEET_REFS}" (at 78.7400 66.0400 0) (effects (font (size 1.016 1.016))  (hide yes))))
+(wire (pts (xy 81.2800 71.1200) (xy 78.7400 71.1200)) (stroke (width 0) (type default)))
+(global_label "female3/mic direct" (shape bidirectional) (at 78.7400 71.1200 180) (effects (font (size 0.95 0.95)) (justify right)) (property "Intersheetrefs" "${INTERSHEET_REFS}" (at 78.7400 71.1200 0) (effects (font (size 1.016 1.016))  (hide yes))))
+(wire (pts (xy 81.2800 76.2000) (xy 78.7400 76.2000)) (stroke (width 0) (type default)))
+(global_label "male1/mic direct" (shape bidirectional) (at 78.7400 76.2000 180) (effects (font (size 0.95 0.95)) (justify right)) (property "Intersheetrefs" "${INTERSHEET_REFS}" (at 78.7400 76.2000 0) (effects (font (size 1.016 1.016))  (hide yes))))
+(wire (pts (xy 81.2800 81.2800) (xy 78.7400 81.2800)) (stroke (width 0) (type default)))
+(global_label "male2/mic direct" (shape bidirectional) (at 78.7400 81.2800 180) (effects (font (size 0.95 0.95)) (justify right)) (property "Intersheetrefs" "${INTERSHEET_REFS}" (at 78.7400 81.2800 0) (effects (font (size 1.016 1.016))  (hide yes))))
 (no_connect (at 81.2800 86.3600))
 (no_connect (at 81.2800 91.4400))
@@
 (wire (pts (xy 287.0200 91.4400) (xy 284.4800 91.4400)) (stroke (width 0) (type default)))
 (global_label "GND" (shape bidirectional) (at 284.4800 91.4400 180) (effects (font (size 0.95 0.95)) (justify right)) (property "Intersheetrefs" "${INTERSHEET_REFS}" (at 284.4800 91.4400 0) (effects (font (size 1.016 1.016))  (hide yes))))
-(wire (pts (xy 287.0200 96.5200) (xy 284.4800 96.5200)) (stroke (width 0) (type default)))
-(global_label "IOREF" (shape bidirectional) (at 284.4800 96.5200 180) (effects (font (size 0.95 0.95)) (justify right)) (property "Intersheetrefs" "${INTERSHEET_REFS}" (at 284.4800 96.5200 0) (effects (font (size 1.016 1.016))  (hide yes))))
+(no_connect (at 287.0200 96.5200))
 (no_connect (at 287.0200 101.6000))
 (no_connect (at 287.0200 106.6800))
