File: CAD/KiCad/shields/voice-active/circuit.kicad_sch (KiCad schematic)
At the start: 10 parts, among them U1 MCP6024-I/SL

Commit message: Route the shield set and validate shared interfaces
Changed lines of the file:
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@@
 (kicad_sch (version 20250114) (generator "eeschema") (generator_version "9.0")
  (paper "A3")
-          (title_block (title "voice-active / circuit") (date "2026-10-01") (rev "A-review")
+          (title_block (title "voice-active / circuit") (date "2026-10-04") (rev "A-prototype")
             (company "Colloquy of Mobiles") (comment 1 "Prototype: verify harness polarity and sensor values before connection"))
           (text "COLLOQUY / VOICE-ACTIVE / CIRCUIT" (at 15.24 15.24 0) (effects (font (size 2.032 2.032) (bold yes)) (justify left top)))

Commit message: Remove shield identification and adopt the simplified connector and Teensy pin maps
Parts:
- removed C1: 470pF C0G, Shields:C_0603_1608Metric, symbol Colloquy:C1
- added C4: 22nF C0G, Shields:C_0805_2012Metric, symbol Colloquy:C4
Connections:
- net stage2/mid: now also C4.1
- net stage2/out: now also C4.2
Other:
- moved on the sheet: C2, C3, R3, R4, R5, R6
