File: CAD/KiCad/shields/backplane/power.kicad_sch (KiCad schematic)
At the start: 11 parts, among them J2 DC jack, J6 screw bridge, J7 JST EH 3, M1 U2D2

Commit message: Update shields for Thomas RC cards, debug headers and body microphones
Parts:
- removed TP31: test pad, Shields:TestPoint_Pad_D1.5mm, symbol Colloquy:TP31
Other:
- moved on the sheet: TP32
Changed lines of the file:
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@@
 (wire (pts (xy 63.5000 215.9000) (xy 60.9600 215.9000)) (stroke (width 0) (type default)))
 (global_label "amp shutdown" (shape bidirectional) (at 60.9600 215.9000 180) (effects (font (size 0.95 0.95)) (justify right)) (property "Intersheetrefs" "${INTERSHEET_REFS}" (at 60.9600 215.9000 0) (effects (font (size 1.016 1.016))  (hide yes))))
-(symbol (lib_id "Colloquy:TP31") (at 195.5800 215.9000 0) (unit 1) (exclude_from_sim no) (in_bom no) (on_board yes) (dnp no)
-(property "Reference" "TP31" (at 200.6600 212.0900 0) (effects (font (size 1.016 1.016))  ))
+(symbol (lib_id "Colloquy:TP32") (at 195.5800 215.9000 0) (unit 1) (exclude_from_sim no) (in_bom no) (on_board yes) (dnp no)
+(property "Reference" "TP32" (at 200.6600 212.0900 0) (effects (font (size 1.016 1.016))  ))
 (property "Value" "test pad" (at 200.6600 214.6300 0) (effects (font (size 1.016 1.016))  ))
 (property "Footprint" "Shields:TestPoint_Pad_D1.5mm" (at 195.5800 215.9000 0) (effects (font (size 1.27 1.27))  (hide yes)))
 (property "Datasheet" "" (at 195.5800 215.9000 0) (effects (font (size 1.27 1.27))  (hide yes)))
-(property "Description" "+5V rail" (at 195.5800 215.9000 0) (effects (font (size 1.27 1.27))  (hide yes)))
-(pin "1")
-(instances (project "backplane" (path "/c974ff16-a701-53ef-8165-966482bbbbae/894454a2-d177-57a2-9ba1-53ccc0188784" (reference "TP31") (unit 1)))))
-(wire (pts (xy 193.0400 215.9000) (xy 190.5000 215.9000)) (stroke (width 0) (type default)))
-(global_label "+5V" (shape bidirectional) (at 190.5000 215.9000 180) (effects (font (size 0.95 0.95)) (justify right)) (property "Intersheetrefs" "${INTERSHEET_REFS}" (at 190.5000 215.9000 0) (effects (font (size 1.016 1.016))  (hide yes))))
-(symbol (lib_id "Colloquy:TP32") (at 325.1200 215.9000 0) (unit 1) (exclude_from_sim no) (in_bom no) (on_board yes) (dnp no)
-(property "Reference" "TP32" (at 330.2000 212.0900 0) (effects (font (size 1.016 1.016))  ))
-(property "Value" "test pad" (at 330.2000 214.6300 0) (effects (font (size 1.016 1.016))  ))
-(property "Footprint" "Shields:TestPoint_Pad_D1.5mm" (at 325.1200 215.9000 0) (effects (font (size 1.27 1.27))  (hide yes)))
-(property "Datasheet" "" (at 325.1200 215.9000 0) (effects (font (size 1.27 1.27))  (hide yes)))
-(property "Description" "MEGA_5V rail" (at 325.1200 215.9000 0) (effects (font (size 1.27 1.27))  (hide yes)))
+(property "Description" "MEGA_5V rail" (at 195.5800 215.9000 0) (effects (font (size 1.27 1.27))  (hide yes)))
 (pin "1")
 (instances (project "backplane" (path "/c974ff16-a701-53ef-8165-966482bbbbae/894454a2-d177-57a2-9ba1-53ccc0188784" (reference "TP32") (unit 1)))))
-(wire (pts (xy 322.5800 215.9000) (xy 320.0400 215.9000)) (stroke (width 0) (type default)))
-(global_label "MEGA_5V" (shape bidirectional) (at 320.0400 215.9000 180) (effects (font (size 0.95 0.95)) (justify right)) (property "Intersheetrefs" "${INTERSHEET_REFS}" (at 320.0400 215.9000 0) (effects (font (size 1.016 1.016))  (hide yes))))
+(wire (pts (xy 193.0400 215.9000) (xy 190.5000 215.9000)) (stroke (width 0) (type default)))
+(global_label "MEGA_5V" (shape bidirectional) (at 190.5000 215.9000 180) (effects (font (size 0.95 0.95)) (justify right)) (property "Intersheetrefs" "${INTERSHEET_REFS}" (at 190.5000 215.9000 0) (effects (font (size 1.016 1.016))  (hide yes))))
           (embedded_fonts no))
