File: CAD/KiCad/shields/backplane/backplane.kicad_pcb (KiCad board)
At the start: 4 copper layers, 210 x 297 mm, 107 parts, among them J1 DSUB-15, J2 DC jack, J5 DSUB-15, J6 screw bridge, J7 JST EH 3, M1 U2D2

Commit message: Remove shield identification and adopt the simplified connector and Teensy pin maps
Parts:
- removed CI1: 10uF X7R, Shields:C_0805_2012Metric
- removed H1, H2, H3, H4: M3 3.2mm NPTH, Shields:MountingHole_3.2mm_M3
- removed RI1, RI2: 4K7, Shields:R_0603_1608Metric
- removed TPI2: shield/sda, Shields:TestPoint_Pad_D1.5mm
- removed TPI3: shield/scl, Shields:TestPoint_Pad_D1.5mm
- added TPA1: female1/analyser out, Shields:TestPoint_Pad_D1.5mm, F.Cu at (100.0, 305.0)
- added TPA2: female2/analyser out, Shields:TestPoint_Pad_D1.5mm, F.Cu at (122.0, 305.0)
- added TPA3: female3/analyser out, Shields:TestPoint_Pad_D1.5mm, F.Cu at (144.0, 305.0)
- added TPA4: male1/analyser out, Shields:TestPoint_Pad_D1.5mm, F.Cu at (166.0, 305.0)
- added TPA5: male2/analyser out, Shields:TestPoint_Pad_D1.5mm, F.Cu at (188.0, 305.0)
- added TPL1: female1/filter out, Shields:TestPoint_Pad_D1.5mm, F.Cu at (90.0, 225.0)
- added TPL2: female2/filter out, Shields:TestPoint_Pad_D1.5mm, F.Cu at (122.0, 225.0)
- added TPL3: female3/filter out, Shields:TestPoint_Pad_D1.5mm, F.Cu at (154.0, 225.0)
- added TPL4: male1/filter out, Shields:TestPoint_Pad_D1.5mm, F.Cu at (186.0, 225.0)
- added TPL5: male2/filter out, Shields:TestPoint_Pad_D1.5mm, F.Cu at (218.0, 225.0)
- added TPM1: female1/microphone, Shields:TestPoint_Pad_D1.5mm, F.Cu at (100.0, 283.0)
- added TPM2: female2/microphone, Shields:TestPoint_Pad_D1.5mm, F.Cu at (122.0, 283.0)
- added TPM3: female3/microphone, Shields:TestPoint_Pad_D1.5mm, F.Cu at (144.0, 283.0)
- added TPM4: male1/microphone, Shields:TestPoint_Pad_D1.5mm, F.Cu at (166.0, 283.0)
- added TPM5: male2/microphone, Shields:TestPoint_Pad_D1.5mm, F.Cu at (188.0, 283.0)
- JA1: value ANALYSER - KEY 24 -> ANALYSER - KEY 22; footprint Shields:Header_2x12_Key24 -> Shields:Header_2x11_Key22
- JV1: value female1 - KEY 14 -> female1 - KEY 6; footprint Shields:Header_2x07_Key14 -> Shields:Header_2x03_Key6
- JV2: value female2 - KEY 14 -> female2 - KEY 6; footprint Shields:Header_2x07_Key14 -> Shields:Header_2x03_Key6
- JV3: value female3 - KEY 14 -> female3 - KEY 6; footprint Shields:Header_2x07_Key14 -> Shields:Header_2x03_Key6
- JV4: value male1 - KEY 14 -> male1 - KEY 6; footprint Shields:Header_2x07_Key14 -> Shields:Header_2x03_Key6
- JV5: value male2 - KEY 14 -> male2 - KEY 6; footprint Shields:Header_2x07_Key14 -> Shields:Header_2x03_Key6
Connections:
- A1 pad SCL: shield/scl -> (no net)
- A1 pad SDA: shield/sda -> (no net)
- JA1 pad 19: shield/sda -> IOREF
- JA1 pad 20: shield/scl -> GND
- JA1 pad 21: IOREF -> +5V
Routing:
- net shield/scl: track 391.1 -> 0.00 mm, vias 6 -> 0
- net shield/sda: track 381.9 -> 0.00 mm, vias 5 -> 0
- net IOREF: track 447.7 -> 338.1 mm, vias 5 -> 3
- net male1/microphone: track 81.5 -> 172.7 mm
- net GND: track 1097.5 -> 1013.5 mm, vias 8 -> 6
- net female3/microphone: track 82.6 -> 131.6 mm, vias 1 -> 2
- net female2/microphone: track 57.8 -> 105.4 mm, vias 0 -> 2
- net analyser/reset: track 290.4 -> 254.4 mm, vias 2 -> 3
- net +5V: track 664.3 -> 629.1 mm
- net female1/tone: track 207.8 -> 175.3 mm
- net AGND: track 555.1 -> 527.0 mm, vias 13 -> 11
- net male2/tone: track 139.2 -> 123.5 mm, vias 2 -> 1
- net male2/analyser out: track 310.5 -> 322.4 mm, vias 1 -> 3
- net female1/analyser out: track 267.1 -> 278.3 mm, vias 0 -> 2
- net analyser/strobe: track 299.5 -> 291.5 mm, vias 2 -> 1
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- removed copper zone on In2.Cu, net +5V
- removed copper zone on B.Cu, net AGND
- removed copper zone on In1.Cu, net GND

Commit message: Finish revised shield routing, printed identification and clean KiCad checks
Parts:
- TP1: value test pad -> male1/filter out
- TP11: value test pad -> male1/analyser out
- TP12: value test pad -> male2/analyser out
- TP13: value test pad -> female1/analyser out
- TP14: value test pad -> female2/analyser out
- TP15: value test pad -> female3/analyser out
- TP2: value test pad -> male2/filter out
- TP20: value test pad -> analyser/strobe
- TP21: value test pad -> analyser/reset
- TP3: value test pad -> female1/filter out
- TP30: value test pad -> amp shutdown
- TP31: value test pad -> +5V
- TP32: value test pad -> MEGA_5V
- TP33: value test pad -> GND
- TP34: value test pad -> AGND
- TP4: value test pad -> female2/filter out
- TP5: value test pad -> female3/filter out
- moved TPM5 39.5 mm to (160.2, 311.1)
- moved TPA5 18.0 mm to (184.6, 322.7)
- moved TPL3 1.30 mm to (153.1, 225.9)
Routing:
- net female3/filter out: track 51.6 -> 50.3 mm
- net male2/microphone: vias 0 -> 1
- net male2/analyser out: vias 3 -> 4
- added copper zone on In2.Cu, net +5V
- added copper zone on B.Cu, net AGND
- added copper zone on In1.Cu, net GND
Other:
- board text added: "1"
- board text added: "1 ANA"
- board text added: "1 LINE"
- board text added: "2 ANA"
- board text added: "2 LINE"
- board text added: "3 ANA"
- board text added: "3 LINE"
- board text added: "4 ANA"
- board text added: "4 LINE"
- board text added: "5 ANA"
- board text added: "5 LINE"
- board text added: "AGND"
- board text added: "AMP SHUTDOWN"
- board text added: "ANA 1"
- board text added: "ANA 2"
- board text added: "ANA 3"
- board text added: "ANA 4"
- board text added: "ANA 5"
- board text added: "AUDIO RTN"
- board text added: "BOARD +5V"
- board text added: "CARD PITCH Hz"
- board text added: "CHANGE A SHIELD ONLY WITH BOTH UNPLUGGED"
- board text added: "COLLOQUY - SHIELD BACKPLANE - REV A"
- board text added: "COMPUTING SLOT MEGA 2560 OR TEENSY ADAPTER"
- board text added: "GND"
- board text added: "IOREF: 5 V = MEGA / 3.3 V = TEENSY"
- board text added: "JA1 - ANALYSER - MSGEQ7 OR DIRECT"
- board text added: "JP1 - ONLY AGND-GND BOND"
- board text added: "JV1 - FEMALE1 MEGA D6 - TEENSY 2"
- board text added: "JV2 - FEMALE2 MEGA D46 - TEENSY 4"
- board text added: "JV3 - FEMALE3 MEGA D10 - TEENSY 5"
- board text added: "JV4 - MALE1 MEGA D11 - TEENSY 6"
- board text added: "JV5 - MALE2 MEGA D5 - TEENSY 28"
- board text added: "KEY <-"
- board text added: "LINE 1"
- board text added: "LINE 2"
- board text added: "LINE 3"
- board text added: "LINE 4"
- board text added: "LINE 5"
- board text added: "LINE OUT"
- board text added: "M3"
- board text added: "MEGA 5V (COMPUTING USB)"
- board text added: "MIC 1"
- board text added: "MIC 2"
- board text added: "MIC 3"
- board text added: "MIC 4"
- board text added: "MIC 5"
- board text added: "MIC ORDER F1 F2 F3 M1 M2 - MODULE N = BODY N"
- board text added: "POWER RACK AND COMPUTING USB TOGETHER"
- board text added: "RESET"
- board text added: "SERVO BUS - 12 V"
- board text added: "SLOT N = BODY N"
- board text added: "STROBE"
- board text added: "TONE 1"
- board text added: "TONE 2"
- board text added: "TONE 3"
- board text added: "TONE 4"
- board text added: "TONE 5"
- board text added: "U2D2"
- board text added: "USB END ^"
- board text removed: "COLLOQUY / SHIELDS / A"
- board text removed: "IOREF: MEGA 5V / TEENSY 3.3V"
- board text removed: "JV1 female1"
- board text removed: "JV2 female2"
- board text removed: "JV3 female3"
- board text removed: "JV4 male1"
- board text removed: "JV5 male2"

Commit message: Route microphones directly to Teensy and remove the analyser buffer board
Parts:
- removed TPI1: IOREF, Shields:TestPoint_Pad_D1.5mm
- added RM1: 4K7, Shields:R_0603_1608Metric, F.Cu at (100.0, 289.0)
- added RM2: 4K7, Shields:R_0603_1608Metric, F.Cu at (122.0, 289.0)
- added RM3: 4K7, Shields:R_0603_1608Metric, F.Cu at (144.0, 289.0)
- added RM4: 4K7, Shields:R_0603_1608Metric, F.Cu at (166.0, 289.0)
- added RM5: 4K7, Shields:R_0603_1608Metric, F.Cu at (184.0, 289.0)
- added RMD1: 1M, Shields:R_0603_1608Metric, F.Cu at (104.0, 292.0)
- added RMD2: 1M, Shields:R_0603_1608Metric, F.Cu at (126.0, 292.0)
- added RMD3: 1M, Shields:R_0603_1608Metric, F.Cu at (148.0, 292.0)
- added RMD4: 1M, Shields:R_0603_1608Metric, F.Cu at (170.0, 292.0)
- added RMD5: 1M, Shields:R_0603_1608Metric, F.Cu at (184.0, 293.0)
- added TPD1: female1/mic direct, Shields:TestPoint_Pad_D1.5mm, F.Cu at (100.0, 296.0)
- added TPD2: female2/mic direct, Shields:TestPoint_Pad_D1.5mm, F.Cu at (122.0, 296.0)
- added TPD3: female3/mic direct, Shields:TestPoint_Pad_D1.5mm, F.Cu at (144.0, 296.0)
- added TPD4: male1/mic direct, Shields:TestPoint_Pad_D1.5mm, F.Cu at (166.0, 296.0)
- added TPD5: male2/mic direct, Shields:TestPoint_Pad_D1.5mm, F.Cu at (184.0, 298.0)
Connections:
- A1 pad D26: (no net) -> female1/mic direct
- A1 pad D27: (no net) -> female2/mic direct
- A1 pad D28: (no net) -> female3/mic direct
- A1 pad D29: (no net) -> male1/mic direct
- A1 pad D30: (no net) -> male2/mic direct
- A1 pad IORF: IOREF -> (no net)
- JA1 pad 19: IOREF -> MEGA_5V
- JA1 pad 21: +5V -> GND
Routing:
- net IOREF: track 338.1 -> 0.00 mm, vias 3 -> 0
- net female1/mic direct: track 0.00 -> 216.4 mm, vias 0 -> 2
- net female2/mic direct: track 0.00 -> 202.5 mm, vias 0 -> 2
- net MEGA_5V: track 183.2 -> 357.2 mm, vias 4 -> 5
- net female3/mic direct: track 0.00 -> 172.1 mm, vias 0 -> 1
- net male2/mic direct: track 0.00 -> 168.8 mm, vias 0 -> 2
- net male1/mic direct: track 0.00 -> 165.2 mm, vias 0 -> 1
- net male2/analyser out: track 322.4 -> 446.4 mm, vias 4 -> 2
- net AGND: track 527.0 -> 625.9 mm, vias 11 -> 15
- net male2/photosensor/B: track 300.7 -> 229.2 mm, vias 3 -> 2
- net male2/photosensor/A: track 289.3 -> 230.6 mm, vias 3 -> 2
- net male2/microphone: track 140.1 -> 184.9 mm, vias 1 -> 3
- net +12V: track 399.8 -> 437.2 mm
- net analyser/reset: track 254.4 -> 279.6 mm, vias 3 -> 4
- net dxl_data: track 439.8 -> 417.1 mm
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Other:
- board text added: "JA1 - MSGEQ7 ANALYSER - MEGA ONLY - EMPTY WITH TEENSY"
- board text added: "MIC DIRECT - 4.7 K - TO TEENSY A0-A4"
- board text added: "MIC DIRECT 1"
- board text added: "MIC DIRECT 2"
- board text added: "MIC DIRECT 3"
- board text added: "MIC DIRECT 4"
- board text added: "MIC DIRECT 5"
- board text removed: "IOREF: 5 V = MEGA / 3.3 V = TEENSY"
- board text removed: "JA1 - ANALYSER - MSGEQ7 OR DIRECT"

Commit message: Update shields for Thomas RC cards, debug headers and body microphones
Parts:
- removed TP11: male1/analyser out, Shields:TestPoint_Pad_D1.5mm
- removed TP12: male2/analyser out, Shields:TestPoint_Pad_D1.5mm
- removed TP13: female1/analyser out, Shields:TestPoint_Pad_D1.5mm
- removed TP14: female2/analyser out, Shields:TestPoint_Pad_D1.5mm
- removed TP15: female3/analyser out, Shields:TestPoint_Pad_D1.5mm
- added DP12: GREEN LED, Shields:LED_0603_1608Metric, F.Cu at (217.0, 84.0)
- added DP5: GREEN LED, Shields:LED_0603_1608Metric, F.Cu at (210.0, 84.0)
- added DPUSB: GREEN LED, Shields:LED_0603_1608Metric, F.Cu at (224.0, 84.0)
- added DT1: YELLOW LED, Shields:LED_0603_1608Metric, F.Cu at (82.5, 194.0)
- added DT2: YELLOW LED, Shields:LED_0603_1608Metric, F.Cu at (113.0, 194.0)
- added DT3: YELLOW LED, Shields:LED_0603_1608Metric, F.Cu at (143.5, 194.0)
- added DT4: YELLOW LED, Shields:LED_0603_1608Metric, F.Cu at (174.0, 194.0)
- added DT5: YELLOW LED, Shields:LED_0603_1608Metric, F.Cu at (204.5, 194.0)
- added RLP12: 4K7, Shields:R_0603_1608Metric, F.Cu at (217.0, 87.0)
- added RLP5: 2K2, Shields:R_0603_1608Metric, F.Cu at (210.0, 87.0)
- added RLPUSB: 2K2, Shields:R_0603_1608Metric, F.Cu at (224.0, 87.0)
- added RLT1: 1K5, Shields:R_0603_1608Metric, F.Cu at (82.5, 197.0)
- added RLT2: 1K5, Shields:R_0603_1608Metric, F.Cu at (113.0, 197.0)
- added RLT3: 1K5, Shields:R_0603_1608Metric, F.Cu at (143.5, 197.0)
- added RLT4: 1K5, Shields:R_0603_1608Metric, F.Cu at (174.0, 197.0)
- added RLT5: 1K5, Shields:R_0603_1608Metric, F.Cu at (204.5, 197.0)
- added TPEG: AGND, Shields:TestPin_1x01_P2.54mm, F.Cu at (151.6, 322.0)
- added TPUSB: MEGA_5V, Shields:TestPin_1x01_P2.54mm, F.Cu at (221.2, 93.0)
- added TPVG: AGND, Shields:TestPin_1x01_P2.54mm, F.Cu at (222.2, 202.0)
- TP31, TPA1, TPA2, TPA3, TPA4, TPA5, TPD1, TPD2, TPD3, TPD4, TPD5, TPL1, TPL2, TPL3, TPL4, TPL5, TPV1, TPV2, TPV3, TPV4, TPV5: footprint Shields:TestPoint_Pad_D1.5mm -> Shields:TestPin_1x01_P2.54mm
- TP33: value GND -> +12V; footprint Shields:TestPoint_Pad_D1.5mm -> Shields:TestPin_1x01_P2.54mm
- TP34: value AGND -> GND; footprint Shields:TestPoint_Pad_D1.5mm -> Shields:TestPin_1x01_P2.54mm
- moved TP34 116.8 mm to (223.7, 93.0)
- moved TPD5 51.1 mm to (138.9, 322.0)
- moved TPD4 45.4 mm to (128.8, 322.0)
- moved TPA5 43.1 mm to (141.5, 322.0)
- moved TPA4 38.6 mm to (131.3, 322.0)
- moved TPD3 36.3 mm to (118.6, 322.0)
- moved TPD2 29.3 mm to (108.5, 322.0)
- moved TPA3 28.5 mm to (121.2, 322.0)
- moved TPD1 26.1 mm to (98.3, 322.0)
- moved TPL5 25.5 mm to (207.0, 202.0)
- moved TPL3 24.9 mm to (146.0, 202.0)
- moved TPL4 24.9 mm to (176.5, 202.0)
- moved TPL2 23.9 mm to (115.6, 202.0)
- moved TPL1 23.5 mm to (85.1, 202.0)
- moved TP31 22.7 mm to (211.0, 93.0)
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Connections:
- TP33 pad 1: GND -> +12V
- TP34 pad 1: AGND -> GND
Routing:
- net +12V: track 437.2 -> 590.9 mm
- net male2/analyser out: track 446.4 -> 296.9 mm, vias 2 -> 0
- net GND: track 1027.1 -> 1099.6 mm, vias 7 -> 11
- net MEGA_5V: track 357.2 -> 413.1 mm, vias 5 -> 4
- net female3/mic direct: track 172.1 -> 219.3 mm, vias 1 -> 3
- net male2/mic direct: track 168.8 -> 216.0 mm, vias 2 -> 3
- net female1/mic direct: track 216.4 -> 257.7 mm
- net male1/mic direct: track 165.2 -> 204.0 mm
- net female2/mic direct: track 202.5 -> 232.9 mm, vias 2 -> 3
- net female1/tone: track 179.0 -> 208.9 mm, vias 3 -> 1
- net female2/tone: track 91.2 -> 119.3 mm, vias 2 -> 1
- net male1/analyser out: track 305.5 -> 282.5 mm, vias 5 -> 0
- net male1/photosensor/C: track 281.5 -> 302.6 mm, vias 1 -> 2
- net female3/tone: track 147.4 -> 168.3 mm
- net male1/neopixel: track 265.4 -> 284.0 mm, vias 2 -> 3
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Other:
- board text added: "12V"
- board text added: "5V"
- board text added: "A1"
- board text added: "A2"
- board text added: "A3"
- board text added: "A4"
- board text added: "A5"
- board text added: "BOARD 5V"
- board text added: "L1"
- board text added: "L2"
- board text added: "L3"
- board text added: "L4"
- board text added: "L5"
- board text added: "M1"
- board text added: "M2"
- board text added: "M4"
- board text added: "M5"
- board text added: "MEGA 5V"
- board text added: "T = TONE / L = LINE"
- board text added: "T1"
- board text added: "T2"
- board text added: "T3"
- board text added: "T4"
- board text added: "T5"
- board text added: "USB"
- board text removed: "1 ANA"
- board text removed: "2 ANA"
- board text removed: "3 ANA"
- board text removed: "4 ANA"
- board text removed: "5 ANA"
- board text removed: "ANA 1"
- board text removed: "ANA 2"
- board text removed: "ANA 3"
- board text removed: "ANA 4"
- board text removed: "ANA 5"
- board text removed: "BOARD +5V"
- board text removed: "LINE 1"
- board text removed: "LINE 2"
- board text removed: "LINE 3"
- board text removed: "LINE 4"
- board text removed: "LINE 5"
- board text removed: "MIC DIRECT 1"
- board text removed: "MIC DIRECT 2"
- board text removed: "MIC DIRECT 3"
- board text removed: "MIC DIRECT 4"
- board text removed: "MIC DIRECT 5"
- board text removed: "SLOT N = BODY N"

Commit message: Move the computing slot to the front and widen outer servo power routing
Parts:
- A1: footprint Shields:Arduino_Mega2560_R3_Shield -> Shields:Mega_Front_Mirrored
- HM1, HM2, HM3, HM4: value M3 computing shield -> M3; front spacer OD <=4mm; screw head on rear; footprint Shields:MountingHole_3.2mm_M3 -> Shields:MountingHole_3.2mm_M3_SlimFront
- moved A1 53.3 mm to (194.5, 53.3)
- moved HM1 48.3 mm to (192.0, 149.8)
- moved HM2 48.3 mm to (143.7, 68.6)
- moved HM3 48.3 mm to (143.7, 143.5)
- moved HM4 48.3 mm to (192.0, 67.3)
Routing:
- net MEGA_5V: track 413.1 -> 327.7 mm, vias 4 -> 3
- net female2/analyser out: track 258.3 -> 325.3 mm, vias 1 -> 2
- net GND: track 1099.6 -> 1160.6 mm, vias 11 -> 13
- net female1/analyser out: track 279.0 -> 335.5 mm
- net female3/analyser out: track 282.8 -> 339.1 mm, vias 0 -> 1
- net female1/mic direct: track 257.7 -> 202.2 mm, vias 2 -> 1
- net male2/tone: track 128.8 -> 183.8 mm, vias 0 -> 2
- net female1/photosensor: track 260.0 -> 312.6 mm
- net female2/neopixel/driven: track 49.8 -> 100.2 mm
- net female1/neopixel/driven: track 23.9 -> 72.2 mm
- net male2/neopixel/driven: track 36.5 -> 84.6 mm
- net amp shutdown: track 22.6 -> 70.5 mm
- net male1/bar neopixel/driven: track 39.0 -> 85.7 mm
- net male2/bar neopixel/driven: track 41.4 -> 85.9 mm
- net female3/neopixel/driven: track 55.7 -> 99.1 mm, vias 1 -> 2
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Other:
- board text added: "COMPUTING SLOT MEGA 2560 OR TEENSY ADAPTER MEGA COMPONENT SIDE DOWN"
- board text removed: "COMPUTING SLOT MEGA 2560 OR TEENSY ADAPTER"

Commit message: Restore the original enclosure holes in the backplane
Parts:
- moved TPL3 6.43 mm to (141.0, 206.0)
Routing:
- net GND: track 1160.6 -> 1135.5 mm
- net AGND: track 669.1 -> 674.7 mm
- net female3/filter out: track 65.1 -> 61.9 mm
- net +12V: track 568.1 -> 570.9 mm
Other:
- outline, holes or cut-outs redrawn
