File: CAD/KiCad/shields/analyser-carrier/interface.kicad_sch (KiCad schematic)
At the start: 5 parts

Commit message: Convert analyser carrier to direct sockets for modified DFRobot modules
Parts:
- JA1: footprint Shields:Socket_2x11_Key22 -> Shields:Socket_2x11_Key22_PlugCarrier
Changed lines of the file:
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@@
 (property "Reference" "JA1" (at 101.6000 48.2600 0) (effects (font (size 1.016 1.016))  ))
 (property "Value" "ANALYSER - KEY 22" (at 101.6000 50.8000 0) (effects (font (size 1.016 1.016))  ))
-(property "Footprint" "Shields:Socket_2x11_Key22" (at 101.6000 83.8200 0) (effects (font (size 1.27 1.27))  (hide yes)))
+(property "Footprint" "Shields:Socket_2x11_Key22_PlugCarrier" (at 101.6000 83.8200 0) (effects (font (size 1.27 1.27))  (hide yes)))
 (property "Datasheet" "" (at 101.6000 83.8200 0) (effects (font (size 1.27 1.27))  (hide yes)))
 (property "Description" "" (at 101.6000 83.8200 0) (effects (font (size 1.27 1.27))  (hide yes)))
