File: CAD/KiCad/shields/gf1002-reference/gf1002-reference.kicad_pcb (KiCad board)
At the start: 2 copper layers, 20 x 30 mm, 10 parts, among them P1 R_0805_2012Metric, P2 R_0805_2012Metric, P3 R_0805_2012Metric, P4 R_0805_2012Metric, P5 R_0805_2012Metric, P6 R_0805_2012Metric, U1 PHOTO REFERENCE

Commit message: Keep the GF1002 contact row clear on both body boards
Correct the reference to nine contacts on the long edge. Move H2 to the short end, move hookup pads alongside the row, clear nearby components and require flush-cut pin tails. Preserve artwork outlines, DSUB geometry and harness pin order.

Refresh routed PCBs, STEP/VRML models, body scenes, production Gerbers and actual-size templates. User approved the documented dimensional estimates; physical fit and ROUT polarity remain checks before ordering. Native ERC/DRC/parity and clearance checks pass; all 1796 pytest tests pass.
Other:
- board size 20 x 30 mm -> 20.2 x 30 mm
- board text added: "G IN"
- board text added: "L IN"
- board text added: "LOUT A"
- board text added: "LOUT B"
- board text added: "R IN"
- board text added: "ROUT A"
- board text added: "ROUT B"
- board text added: "V+"
- board text added: "V-"
