File: CAD/KiCad/male static v2/male-static-v2.kicad_sch (KiCad schematic)
At the start: 19 parts, among them J1 photosensor, J10 State LED, J11 bar neopixel, J2 dxl male, J3 microphone, J4 photosensor, J5 body neopixel, J6 Speaker, J7 DA15_Plug_MountingHoles, J8 photosensor, J9 photosensor, M1 GF1002 direct module

Commit message: Keep the GF1002 contact row clear on both body boards
Correct the reference to nine contacts on the long edge. Move H2 to the short end, move hookup pads alongside the row, clear nearby components and require flush-cut pin tails. Preserve artwork outlines, DSUB geometry and harness pin order.

Refresh routed PCBs, STEP/VRML models, body scenes, production Gerbers and actual-size templates. User approved the documented dimensional estimates; physical fit and ROUT polarity remain checks before ordering. Native ERC/DRC/parity and clearance checks pass; all 1796 pytest tests pass.
Parts:
- H2: footprint Body:GF1002_Clamp_Right -> Body:GF1002_Clamp_End
Other:
- note added: "JA1: 1=5V, 2=GND, 3=R INPUT, 4=Audio GND, 5=ROUT+, 6=ROUT-. Verify ROUT polarity on module."
- note removed: "JA1: 1=5V, 2=GND, 3=Audio, 4=Audio GND, 5=ROUT+, 6=ROUT-. Module contact positions unverified."
Changed lines of the file:
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@@
 (kicad_sch (version 20250114) (generator "eeschema") (generator_version "9.0")
  (paper "A3")
-          (title_block (title "Colloquy male static — directly mounted GF1002") (date "2026-10-09") (rev "B-direct-amplifier")
+          (title_block (title "Colloquy male static — directly mounted GF1002") (date "2026-10-19") (rev "C-contact-clearance")
             (company "Colloquy of Mobiles") (comment 1 "Prototype: verify harness polarity and sensor values before connection"))
           (text "V2 ENGINEERING PROTOTYPE / DIRECT GF1002 / NO PERFBOARD" (at 15 12 0) (effects (font (size 2 2) (bold yes)) (justify left top)))
 (text "Harness speaker pair becomes LINE_IN / AUDIO_RETURN. Rack must be converted first." (at 15 20 0) (effects (font (size 1.27 1.27) ) (justify left top)))
-(text "JA1: 1=5V, 2=GND, 3=Audio, 4=Audio GND, 5=ROUT+, 6=ROUT-. Module contact positions unverified." (at 15 26 0) (effects (font (size 1.27 1.27) ) (justify left top)))
+(text "JA1: 1=5V, 2=GND, 3=R INPUT, 4=Audio GND, 5=ROUT+, 6=ROUT-. Verify ROUT polarity on module." (at 15 26 0) (effects (font (size 1.27 1.27) ) (justify left top)))
 (text "Insulating edge clamps: do not drill the module. Only harness +5V feeds the amplifier; 12V remains servo-only." (at 15 32 0) (effects (font (size 1.27 1.27) ) (justify left top)))
 (symbol (lib_id "Colloquy:J7") (at 44.4500 110.4900 0) (unit 1) (exclude_from_sim no) (in_bom yes) (on_board yes) (dnp no)
@@
 (property "Footprint" "Body:GF1002_WirePads_2x03" (at 335.2800 59.6900 0) (effects (font (size 1.27 1.27))  (hide yes)))
 (property "Datasheet" "" (at 335.2800 59.6900 0) (effects (font (size 1.27 1.27))  (hide yes)))
-(property "Description" "Short individually identified wires to module VDD, supply GND, Audio, input GND, ROUT+, ROUT-. Pad order is carrier-defined; verify module contacts." (at 335.2800 59.6900 0) (effects (font (size 1.27 1.27))  (hide yes)))
+(property "Description" "Short wires to module VDD, supply GND, R input, input GND, ROUT+, ROUT-. Verify output pair polarity on the actual module; photo does not establish it." (at 335.2800 59.6900 0) (effects (font (size 1.27 1.27))  (hide yes)))
 (pin "1")
 (pin "2")
@@
 (property "Footprint" "Body:GF1002_Module_Direct" (at 340.3600 275.5900 0) (effects (font (size 1.27 1.27))  (hide yes)))
 (property "Datasheet" "" (at 340.3600 275.5900 0) (effects (font (size 1.27 1.27))  (hide yes)))
-(property "Description" "No perfboard. Photo-derived 20x30mm module, held by two insulating edge clamps; 3mm underside clearance." (at 340.3600 275.5900 0) (effects (font (size 1.27 1.27))  (hide yes)))
+(property "Description" "No perfboard. Provisional 20.2x30mm envelope; shaft-edge and short-end insulating clamps. Cut module pin tails flush; 3mm underside gap. Physical fit unverified." (at 340.3600 275.5900 0) (effects (font (size 1.27 1.27))  (hide yes)))
 (instances (project "male-static-v2" (path "/3c3a1eba-aee4-5f63-9472-4e4300e66b7a" (reference "M1") (unit 1)))))
 (symbol (lib_id "Colloquy:H1") (at 240.0300 275.5900 0) (unit 1) (exclude_from_sim no) (in_bom no) (on_board yes) (dnp no)
@@
 (property "Reference" "H2" (at 289.5600 260.3500 0) (effects (font (size 1.016 1.016))  ))
 (property "Value" "M2 insulating clamp" (at 289.5600 262.8900 0) (effects (font (size 1.016 1.016))  ))
-(property "Footprint" "Body:GF1002_Clamp_Right" (at 289.5600 275.5900 0) (effects (font (size 1.27 1.27))  (hide yes)))
+(property "Footprint" "Body:GF1002_Clamp_End" (at 289.5600 275.5900 0) (effects (font (size 1.27 1.27))  (hide yes)))
 (property "Datasheet" "" (at 289.5600 275.5900 0) (effects (font (size 1.27 1.27))  (hide yes)))
 (property "Description" "Provisional edge clamp. No drilling of amplifier module; check actual fit." (at 289.5600 275.5900 0) (effects (font (size 1.27 1.27))  (hide yes)))

Commit message: Socket and reroute the body amplifiers to revision D
Replace JA1 wires with eleven-pin GF1002 sockets, explicit unused contacts and an 11 mm header stack. Move the divider and bypass beside their socket pins, shorten and pair the speaker routes, and separate them from audio and sensor inputs with a grounded guard. Add adjustable support models and preserve the artwork outline, DSUB geometry and harness pin order.

Regenerate schematics, routing, models, current body scenes, Gerbers and actual-size templates. Native ERC/DRC/unconnected/parity are zero on both boards; independent socket, support, decoupling and routing checks pass; all 1796 pytest tests pass. Module fit, purchased stack height, module ground bond and ROUT polarity remain physical checks before ordering.
Parts:
- removed JA1: GF1002 wire connections, Body:GF1002_WirePads_2x03, symbol Colloquy:JA1
- H1: value M2 insulating clamp -> M2 insulating support / 11mm; footprint Body:GF1002_Clamp_Left -> Body:GF1002_Support_Left
- H2: value M2 insulating clamp -> M2 insulating support / 11mm; footprint Body:GF1002_Clamp_End -> Body:GF1002_Support_End
- M1: value GF1002 direct module -> GF1002 / 1x11 female socket; footprint Body:GF1002_Module_Direct -> Body:GF1002_PlugIn_1x11
Connections:
- net 5V: now also M1.5 (VDD)
- net AMP_INPUT: now also M1.1 (R_IN)
- net AMP_OUT_N: now also M1.11 (ROUT_N_VERIFY)
- net AMP_OUT_P: now also M1.10 (ROUT_P_VERIFY)
- net AUDIO_RETURN: now also M1.2 (INPUT_G)
- net GND: now also M1.6 (SUPPLY_GND)
- no-connect marks 1 -> 6
Other:
- note added: "M1: 1=R IN, 2=audio return, 5=5V, 6=GND, 10/11=ROUT+/-. Verify output polarity and ground bond on module."
- note added: "No output is grounded. Audio return and supply ground meet only on the module. Insulating adjustable supports."
- note added: "REV D ENGINEERING PROTOTYPE / SOCKETED GF1002 / 11mm NOMINAL STACK"
- note removed: "Insulating edge clamps: do not drill the module. Only harness +5V feeds the amplifier; 12V remains servo-only."
- note removed: "JA1: 1=5V, 2=GND, 3=R INPUT, 4=Audio GND, 5=ROUT+, 6=ROUT-. Verify ROUT polarity on module."
- note removed: "V2 ENGINEERING PROTOTYPE / DIRECT GF1002 / NO PERFBOARD"
- moved on the sheet: C1, C2, R1, R2

Commit message: Use SMD reservoir capacitors on both v2 body boards
Parts:
- C1: footprint Capacitor_THT:CP_Radial_D6.3mm_P2.50mm -> Capacitor_SMD:CP_Elec_6.3x5.8
Changed lines of the file:
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@@
 (property "Reference" "C1" (at 340.3600 140.9700 0) (effects (font (size 1.016 1.016)) (justify left) ))
 (property "Value" "220uF 10V / provisional" (at 340.3600 143.5100 0) (effects (font (size 1.016 1.016)) (justify left) ))
-(property "Footprint" "Capacitor_THT:CP_Radial_D6.3mm_P2.50mm" (at 335.2800 143.5100 0) (effects (font (size 1.27 1.27))  (hide yes)))
+(property "Footprint" "Capacitor_SMD:CP_Elec_6.3x5.8" (at 335.2800 143.5100 0) (effects (font (size 1.27 1.27))  (hide yes)))
 (property "Datasheet" "" (at 335.2800 143.5100 0) (effects (font (size 1.27 1.27))  (hide yes)))
 (property "Description" "Provisional local reservoir; verify actual amplifier transients and rail sag before release." (at 335.2800 143.5100 0) (effects (font (size 1.27 1.27))  (hide yes)))
