File: CAD/KiCad/shields/teensy-adapter/wired/teensy-adapter-wired.kicad_sch (KiCad schematic)
At the start: 81 parts, among them U1 SN74LV4T125PWR, U2 SN74LV4T125PWR, U3 SN74LV4T125PWR, U4 SN74LV4T125PWR

Commit message: Name the Teensy signals at the GPIOs and on the back silkscreen
Parts:
- added unit 6 of JT2
Connections:
- net at CA38.1, RA38.2, RB38.1: now also JT2.19 (38); no longer JT2.19 (38)
- net at CA39.1, RA39.2, RB39.1: now also JT2.18 (39); no longer JT2.18 (39)
Other:
- note added: "GPIO 10 | m1/neopixel"
- note added: "GPIO 11 | m2/neopixel"
- note added: "GPIO 12 | m2/bar/neopixel"
- note added: "GPIO 14 / A0 | f1/microphone"
- note added: "GPIO 15 / A1 | f2/microphone"
- note added: "GPIO 16 / A2 | f3/microphone"
- note added: "GPIO 17 / A3 | m1/microphone"
- note added: "GPIO 18 / A4 | m2/microphone"
- note added: "GPIO 19 / ADC | f1/photosensor"
- note added: "GPIO 2 | f1/tone"
- note added: "GPIO 20 / ADC | f2/photosensor"
- note added: "GPIO 21 / ADC | f3/photosensor"
- note added: "GPIO 22 / ADC | m1/photosensor/A"
- note added: "GPIO 23 / ADC | m1/photosensor/B"
- note added: "GPIO 24 / ADC | m1/photosensor/C"
- note added: "GPIO 25 / ADC | m1/photosensor/D"
- note added: "GPIO 26 / ADC | m2/photosensor/A"
- note added: "GPIO 27 / ADC | m2/photosensor/B"
- note added: "GPIO 28 | m2/tone"
- note added: "GPIO 29 | m1/bar/neopixel"
- note added: "GPIO 30 | m1/aux"
- note added: "GPIO 31 | m2/aux"
- note added: "GPIO 32 | amp/shutdown"
- note added: "GPIO 38 / ADC | m2/photosensor/C"
- note added: "GPIO 39 / ADC | m2/photosensor/D"
- note added: "GPIO 4 | f2/tone"
- note added: "GPIO 5 | f3/tone"
- note added: "GPIO 6 | m1/tone"
- note added: "GPIO 7 | f1/neopixel"
- note added: "GPIO 8 | f2/neopixel"
- note added: "GPIO 9 | f3/neopixel"
- note added: "amp/shutdown"
- note added: "f1-f3 = female 1-3; m1-m2 = male 1-2. Wire captions are plain text, not electrical connections."
- note added: "f1/microphone"
- note added: "f1/neopixel"
- note added: "f1/photosensor"
- note added: "f1/tone"
- note added: "f2/microphone"
- note added: "f2/neopixel"
- note added: "f2/photosensor"
- note added: "f2/tone"
- note added: "f3/microphone"
- note added: "f3/neopixel"
- note added: "f3/photosensor"
- note added: "f3/tone"
- note added: "m1/aux"
- note added: "m1/bar/neopixel"
- note added: "m1/microphone"
- note added: "m1/neopixel"
- note added: "m1/photosensor/A"
- note added: "m1/photosensor/B"
- note added: "m1/photosensor/C"
- note added: "m1/photosensor/D"
- note added: "m1/tone"
- note added: "m2/aux"
- note added: "m2/bar/neopixel"
- note added: "m2/microphone"
- note added: "m2/neopixel"
- note added: "m2/photosensor/A"
- note added: "m2/photosensor/B"
- note added: "m2/photosensor/C"
- note added: "m2/photosensor/D"
- note added: "m2/tone"
- note removed: "ADC 19"
- note removed: "ADC 20"
- note removed: "ADC 21"
- note removed: "ADC 22"
- note removed: "ADC 23"
- note removed: "ADC 24"
- note removed: "ADC 25"
- note removed: "ADC 26"
- note removed: "ADC 27"
- note removed: "ADC 38"
- note removed: "ADC 39"
- note removed: "GPIO 10"
- note removed: "GPIO 11"
- note removed: "GPIO 12"
- note removed: "GPIO 2"
- note removed: "GPIO 28"
- note removed: "GPIO 29"
- note removed: "GPIO 30"
- note removed: "GPIO 31"
- note removed: "GPIO 32"
- note removed: "GPIO 4"
- note removed: "GPIO 5"
- note removed: "GPIO 6"
- note removed: "GPIO 7"
- note removed: "GPIO 8"
- note removed: "GPIO 9"
- note removed: "No added parts or connections. Plain text captions identify wires; they do not connect them."
- note removed: "amp shutdown"
- note removed: "female1 / mic direct"
- note removed: "female1 / neopixel"
- note removed: "female1 / photosensor"
- note removed: "female1 / tone"
- note removed: "female2 / mic direct"
- note removed: "female2 / neopixel"
- note removed: "female2 / photosensor"
- note removed: "female2 / tone"
- note removed: "female3 / mic direct"
- note removed: "female3 / neopixel"
- note removed: "female3 / photosensor"
- note removed: "female3 / tone"
- note removed: "male1 / aux driven"
- note removed: "male1 / bar neopixel"
- note removed: "male1 / mic direct"
- note removed: "male1 / neopixel"
- note removed: "male1 / photosensor / A"
- note removed: "male1 / photosensor / B"
- note removed: "male1 / photosensor / C"
- note removed: "male1 / photosensor / D"
- note removed: "male1 / tone"
- note removed: "male2 / aux driven"
- note removed: "male2 / bar neopixel"
- note removed: "male2 / mic direct"
- note removed: "male2 / neopixel"
- note removed: "male2 / photosensor / A"
- note removed: "male2 / photosensor / B"
- note removed: "male2 / photosensor / C"
- note removed: "male2 / photosensor / D"
- note removed: "male2 / tone"

Commit message: Show each 3-to-5 V shifter as one complete chip block
Parts:
- removed unit 5 of U1
- removed unit 2 of U1
- removed unit 3 of U1
- removed unit 4 of U1
- removed unit 4 of U2
- removed unit 2 of U2
- removed unit 3 of U2
- removed unit 5 of U2
- removed unit 2 of U3
- removed unit 4 of U3
- removed unit 5 of U3
- removed unit 3 of U3
- removed unit 4 of U4
- removed unit 2 of U4
- removed unit 5 of U4
- removed unit 3 of U4
- U1: symbol Colloquy:U1 -> Colloquy:3to5V_Shifter_U1
- U2: symbol Colloquy:U2 -> Colloquy:3to5V_Shifter_U2
- U3: symbol Colloquy:U3 -> Colloquy:3to5V_Shifter_U3
- U4: symbol Colloquy:U4 -> Colloquy:3to5V_Shifter_U4
Connections:
- net at CB1.1, CB2.1, CB3.1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: now also U1.14 (VCC), U2.14 (VCC), U3.14 (VCC), U4.14 (VCC)
- net at CA19.2, CA20.2, CA21.2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: now also U1.10 (OE3), U1.13 (OE4), U1.4 (OE2), U1.7 (GND), U2.10 (OE3), U2.13 (OE4), U2.4 (OE2), U2.7 (GND), U3.10 (OE3), U3.13 (OE4), U3.4 (OE2), U3.7 (GND), U4.10 (OE3), U4.12 (A4), U4.13 (OE4), U4.4 (OE2), U4.7 (GND)
- net at JM1.D10: now also U1.8 (Y3)
- net at JM1.D11: now also U1.11 (Y4)
- net at JM1.D14: now also U2.6 (Y2)
- net at JM1.D15: now also U3.6 (Y2)
- net at JM1.D16: now also U3.11 (Y4)
- net at JM1.D17: now also U3.8 (Y3)
- net at JM1.D2: now also U4.8 (Y3)
- net at JM1.D25: now also U4.6 (Y2)
- net at JM1.D46: now also U1.6 (Y2)
- net at JM1.D7: now also U2.8 (Y3)
- net at JM1.D8: now also U2.11 (Y4)
- net at JT1.24 (32), RD32.1: now also U4.9 (A3)
- net at JT1.11 (9), RD9.1: now also U2.12 (A4)
- net at JT1.6 (4), RD4.1: now also U1.5 (A2)
- net at JT1.13 (11), RD11.1: now also U3.5 (A2)
- net at JT1.10 (8), RD8.1: now also U2.9 (A3)
- net at JT1.14 (12), RD12.1: now also U3.9 (A3)
- net at JT1.21 (29), RD29.1: now also U3.12 (A4)
- net at JT1.23 (31), RD31.1: now also U4.5 (A2)
- net at JT1.7 (5), RD5.1: now also U1.9 (A3)
- net at JT1.8 (6), RD6.1: now also U1.12 (A4)
- net at JT1.9 (7), RD7.1: now also U2.5 (A2)
Other:
- note added: "01 DIGITAL OUTPUTS / 3.3 V GPIO -> 3to5V SHIFTERS -> 5 V backplane"
- note added: "3.3 V IN -> 5 V OUT"
- note added: "3to5V_Shifter_1"
- note added: "3to5V_Shifter_2"
- note added: "3to5V_Shifter_3"
- note added: "3to5V_Shifter_4"
- note added: "5 V"
- note added: "5 V supply"
- note added: "SN74LV4T125PWR"
- note added: "Same circuit and PCB pin numbers | One sheet, no electrical net labels | Review copy 21 Oct 2026"
- note added: "U1 / shifter decoupling"
- note added: "U2 / shifter decoupling"
- note added: "U3 / shifter decoupling"
- note added: "U4 / shifter decoupling"
- note added: "Unused channel / input held at GND"
- note removed: "01 DIGITAL OUTPUTS / Teensy -> 5 V buffers -> backplane"
- note removed: "Same circuit and PCB pin numbers | One sheet, no electrical net labels | Review copy 20 Oct 2026"
- note removed: "Unused buffer gate"
- moved on the sheet: JM1A, JT1A, RD10, RD11, RD12, RD2, RD28, RD29, RD30, RD31, RD32, RD4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
