File: CAD/KiCad/proposed-solutions/shields/voice-thomas/circuit.kicad_sch (KiCad schematic)
At the start: 8 parts

Commit message: Resolve PCB order findings before retrying fabrication and assembly
Parts:
- R3: footprint Shields:R_0603_1608Metric -> Shields:R_Axial_DIN0207_L6.3mm_D2.5mm_P7.62mm_Horizontal
Changed lines of the file:
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@@
 (property "Reference" "R3" (at 195.5800 75.1840 0) (effects (font (size 1.016 1.016))  ))
 (property "Value" "100K" (at 195.5800 77.7240 0) (effects (font (size 1.016 1.016))  ))
-(property "Footprint" "Shields:R_0603_1608Metric" (at 195.5800 81.2800 0) (effects (font (size 1.27 1.27))  (hide yes)))
+(property "Footprint" "Shields:R_Axial_DIN0207_L6.3mm_D2.5mm_P7.62mm_Horizontal" (at 195.5800 81.2800 0) (effects (font (size 1.27 1.27))  (hide yes)))
 (property "Datasheet" "" (at 195.5800 81.2800 0) (effects (font (size 1.27 1.27))  (hide yes)))
 (property "Description" "" (at 195.5800 81.2800 0) (effects (font (size 1.27 1.27))  (hide yes)))
